File: circuits/lil_duder/lil_duder.sch (KiCad schematic (older format))
At the start: 61 parts, among them J1 Mic+, J10 GND_Conn, J11 RST+, J12 RST-, J13 LED4, J14 A1, J2 Mic-, J3 LED1, J4 LED2, J5 SPK_A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

Commit message: switched power to 5v for speaker driver
Connections:
- net +5V: now also C5.1, U4.3 (V+)
- net +9V: no longer C5.1, U4.3 (V+)
Changed lines of the file:
@@
-$EndComp
-$Comp
-L power:+9V #PWR027
-U 1 1 619C2C38
-P 9750 5600
-F 0 "#PWR027" H 9750 5450 50  0001 C CNN
-F 1 "+9V" H 9765 5773 50  0000 C CNN
-F 2 "" H 9750 5600 50  0001 C CNN
-F 3 "" H 9750 5600 50  0001 C CNN
-	1    9750 5600
-	1    0    0    -1
 $EndComp
 $Comp
@@
 Wire Wire Line
 	9650 4950 9650 5000
-Connection ~ 9750 5600
 Wire Wire Line
 	6850 3150 7250 3150
@@
 	1    0    0    -1
 $EndComp
+$Comp
+L power:+5V #PWR?
+U 1 1 618F4DDC
+P 9750 5600
+F 0 "#PWR?" H 9750 5450 50  0001 C CNN
+F 1 "+5V" H 9765 5773 50  0000 C CNN
+F 2 "" H 9750 5600 50  0001 C CNN
+F 3 "" H 9750 5600 50  0001 C CNN
+	1    9750 5600
+	1    0    0    -1
+$EndComp
+Connection ~ 9750 5600
 $EndSCHEMATC

Commit message: changes to circuit
Parts:
- removed R15: 10k, Resistor_THT:R_Axial_DIN0207_L6.3mm_D2.5mm_P7.62mm_Horizontal, symbol Device:R_US
- removed R17: 100k, Resistor_THT:R_Axial_DIN0207_L6.3mm_D2.5mm_P7.62mm_Horizontal, symbol Device:R_US
Connections:
- net Earth: now also U2.5 (+)
- net at R4.1, U2.1: now also U1.23 (PC0)
- net at R3.1, U2.3 (+): no longer U2.5 (+)
- net at U2.6 (-): now also U2.7
Other:
- moved on the sheet: U2B
Changed lines of the file:
@@
 L Amplifier_Operational:TL072 U2
 U 2 1 61829A70
-P 4700 6050
-F 0 "U2" H 4700 6300 50  0000 C CNN
-F 1 "TL072" H 4800 6200 50  0000 C CNN
-F 2 "Package_DIP:DIP-8_W7.62mm_Socket" H 4700 6050 50  0001 C CNN
-F 3 "http://www.ti.com/lit/ds/symlink/tl071.pdf" H 4700 6050 50  0001 C CNN
-	2    4700 6050
+P 4900 6050
+F 0 "U2" H 4900 6300 50  0000 C CNN
+F 1 "TL072" H 5000 6200 50  0000 C CNN
+F 2 "Package_DIP:DIP-8_W7.62mm_Socket" H 4900 6050 50  0001 C CNN
+F 3 "http://www.ti.com/lit/ds/symlink/tl071.pdf" H 4900 6050 50  0001 C CNN
+	2    4900 6050
 	1    0    0    1
 $EndComp
@@
 	1    0    0    -1
 $EndComp
-$Comp
-L Device:R_US R15
-U 1 1 618AB20A
-P 4250 5950
-F 0 "R15" V 4045 5950 50  0000 C CNN
-F 1 "10k" V 4136 5950 50  0000 C CNN
-F 2 "Resistor_THT:R_Axial_DIN0207_L6.3mm_D2.5mm_P7.62mm_Horizontal" V 4290 5940 50  0001 C CNN
-F 3 "~" H 4250 5950 50  0001 C CNN
-	1    4250 5950
-	0    1    1    0
-$EndComp
-Connection ~ 4100 5950
-$Comp
-L Device:R_US R17
-U 1 1 618AB96A
-P 4700 5700
-F 0 "R17" V 4495 5700 50  0000 C CNN
-F 1 "100k" V 4586 5700 50  0000 C CNN
-F 2 "Resistor_THT:R_Axial_DIN0207_L6.3mm_D2.5mm_P7.62mm_Horizontal" V 4740 5690 50  0001 C CNN
-F 3 "~" H 4700 5700 50  0001 C CNN
-	1    4700 5700
-	0    1    1    0
-$EndComp
-Wire Wire Line
-	4550 5700 4400 5700
-Wire Wire Line
-	4400 5700 4400 5950
-Connection ~ 4400 5950
-Wire Wire Line
-	4850 5700 5000 5700
-Wire Wire Line
-	5000 5700 5000 6050
-Wire Wire Line
-	4100 5250 5000 5250
-Wire Wire Line
-	5000 5250 5000 5700
-Connection ~ 5000 5700
+Wire Wire Line
+	4600 5700 4600 5950
+Wire Wire Line
+	5200 5700 5200 6050
 Wire Wire Line
 	4600 3700 4600 3750
@@
 Wire Wire Line
 	2900 2900 4100 2900
-Wire Wire Line
-	4100 2900 4100 5250
 $Comp
 L Device:R_US R14
@@
 	3400 6050 3400 6450
 Wire Wire Line
-	3400 6450 4400 6450
-Wire Wire Line
-	4400 6450 4400 6150
-Connection ~ 3400 6450
+	4600 6450 4600 6150
 Wire Notes Line
 	5300 7050 1950 7050
@@
 $EndComp
 $Comp
-L power:+5V #PWR?
+L power:+5V #PWR029
 U 1 1 618F4DDC
 P 9750 5600
-F 0 "#PWR?" H 9750 5450 50  0001 C CNN
+F 0 "#PWR029" H 9750 5450 50  0001 C CNN
 F 1 "+5V" H 9765 5773 50  0000 C CNN
 F 2 "" H 9750 5600 50  0001 C CNN
@@
 $EndComp
 Connection ~ 9750 5600
+Wire Wire Line
+	4100 2900 4100 5400
+Connection ~ 4100 5400
+Wire Wire Line
+	4600 5700 5200 5700
+$Comp
+L power:Earth #PWR027
+U 1 1 61ABD464
+P 4600 6450
+F 0 "#PWR027" H 4600 6200 50  0001 C CNN
+F 1 "Earth" H 4600 6300 50  0001 C CNN
+F 2 "" H 4600 6450 50  0001 C CNN
+F 3 "~" H 4600 6450 50  0001 C CNN
+	1    4600 6450
+	-1   0    0    -1
+$EndComp
 $EndSCHEMATC
